File: fake-fuko-controller/fake-fuko-controller.kicad_sch (KiCad schematic)
At the start: 16 parts, among them J1 Conn_01x05, J2 Conn_01x02, J3 Conn_01x12, J4 Conn_01x02, U1 ESP32-C3-DEVKITM-1, U3 P78E05-1000

Commit message: Add diode partnos
Parts:
- D1: PartNo (none) -> GS1A_R1_00001
- D2: PartNo (none) -> SMAJ24A-13-F
Changed lines of the file:
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@@
+      (effects (font (size 1.27 1.27)) hide)
+    )
+    (property "Manufacturer" "" (at 44.45 48.26 0)
+      (effects (font (size 1.27 1.27)) hide)
+    )
+    (property "PartNo" "SMAJ24A-13-F" (at 44.45 48.26 0)
       (effects (font (size 1.27 1.27)) hide)
     )
@@
       (effects (font (size 1.27 1.27)) hide)
     )
+    (property "Manufacturer" "" (at 35.56 44.45 0)
+      (effects (font (size 1.27 1.27)) hide)
+    )
+    (property "PartNo" "GS1A_R1_00001" (at 35.56 44.45 0)
+      (effects (font (size 1.27 1.27)) hide)
+    )
